Commit message: add gezebo color and friction coefficient

File: src/my_urdf/description/simple_urdf.xacro (robot description, xacro)
@@ -99,4 +99,9 @@
 		</xacro:inertial_sphere>
 	</link>
+	<gazebo reference="caster_wheel">
+        	<material>Gazebo/Black</material>
+        	<mu1 value="0.001"/>
+        	<mu2 value="0.001"/>
+    	</gazebo>
 	<!--lidar-->
 	<joint name="laser_joint" type="fixed">
